File: SimpleCANBreakout.kicad_pcb (KiCad board)
At the start: 2 copper layers, 31.5 x 15.5 mm, 17 parts, among them U1 TCAN332, U2 AMS1117-3.3

Commit message: Swap TCAN332 for SN65HVD230 and add LCSC part numbers
Rs (pin 8) is tied to GND through the existing pour for high-speed mode.
Production files regenerated with the Fabrication Toolkit.
Parts:
- U1: value TCAN332 -> SN65HVD230
Connections:
- U1 pad 8: unconnected-(U1-NC-Pad8) -> GND
Changed lines of the file:
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@@
+			)
+		)
+		(property "LCSC Part" "C14663"
+			(at 0 0 90)
+			(unlocked yes)
+			(layer "F.Fab")
+			(hide yes)
+			(effects
+				(font
+					(size 1 1)
+					(thickness 0.15)
+				)
 			)
 		)
@@
 			)
 		)
+		(property "LCSC Part" "C14663"
+			(at 0 0 0)
+			(unlocked yes)
+			(layer "F.Fab")
+			(hide yes)
+			(effects
+				(font
+					(size 1 1)
+					(thickness 0.15)
+				)
+			)
+		)
 		(property ki_fp_filters "C_*")
 		(sheetname "/")
@@
 				(font
 					(size 1.27 1.27)
+					(thickness 0.15)
+				)
+			)
+		)
+		(property "LCSC Part" "C6186"
+			(at 0 0 270)
+			(unlocked yes)
+			(layer "F.Fab")
+			(hide yes)
+			(effects
+				(font
+					(size 1 1)
 					(thickness 0.15)
 				)
@@
 			)
 		)
-		(property "Value" "TCAN332"
+		(property "Value" "SN65HVD230"
 			(at 0 3.4 90)
 			(layer "F.Fab")
@@
 			)
 		)
-		(property "Datasheet" "http://www.ti.com/lit/ds/symlink/tcan337.pdf"
-			(at 0 0 90)
-			(layer "F.Fab")
-			(hide yes)
-			(effects
-				(font
-					(size 1.27 1.27)
-				)
-			)
-		)
-		(property "Description" "High-Speed CAN Transceiver, 1Mbps, 3.3V supply, SOT-23-8/SOIC-8"
+		(property "Datasheet" "http://www.ti.com/lit/ds/symlink/sn65hvd230.pdf"
+			(at 0 0 90)
+			(layer "F.Fab")
+			(hide yes)
+			(effects
+				(font
+					(size 1.27 1.27)
+				)
+			)
+		)
+		(property "Description" "CAN Bus Transceivers, 3.3V, 1Mbps, Low-Power capabilities, SOIC-8"
 			(at 0 0 90)
 			(layer "F.Fab")
@@
 			(at 0 0 90)
 			(layer "F.SilkS")
+			(hide yes)
+			(effects
+				(font
+					(size 1 1)
+					(thickness 0.15)
+				)
+			)
+		)
+		(property "LCSC Part" "C12084"
+			(at 0 0 270)
+			(unlocked yes)
+			(layer "F.Fab")
 			(hide yes)
 			(effects
@@
 			(roundrect_rratio 0.25)
 			(net "/CAN TX")
-			(pinfunction "TXD_1")
+			(pinfunction "D_1")
 			(pintype "input")
 		)
@@
 			(roundrect_rratio 0.25)
 			(net "/CAN RX")
-			(pinfunction "RXD_4")
-			(pintype "tri_state")
+			(pinfunction "R_4")
+			(pintype "output")
 		)
 		(pad "5" smd roundrect
@@
 			(layers "F.Cu" "F.Mask" "F.Paste")
 			(roundrect_rratio 0.25)
-			(net "unconnected-(U1-NC-Pad5)")
-			(pinfunction "NC_5")
-			(pintype "no_connect")
+			(net "unconnected-(U1-Vref-Pad5)")
+			(pinfunction "Vref_5")
+			(pintype "output+no_connect")
 		)
 		(pad "6" smd roundrect
@@
 			(layers "F.Cu" "F.Mask" "F.Paste")
 			(roundrect_rratio 0.25)
-			(net "unconnected-(U1-NC-Pad8)")
-			(pinfunction "NC_8")
-			(pintype "no_connect")
+			(net "GND")
+			(pinfunction "Rs_8")
+			(pintype "input")
 		)
 		(embedded_fonts no)
@@
 			(at 0 0 90)
 			(layer "F.SilkS")
+			(hide yes)
+			(effects
+				(font
+					(size 1 1)
+					(thickness 0.15)
+				)
+			)
+		)
+		(property "LCSC Part" "C22787"
+			(at 0 0 270)
+			(unlocked yes)
+			(layer "F.Fab")
 			(hide yes)
 			(effects
@@
 			)
 		)
+		(property "LCSC Part" "C14663"
+			(at 0 0 270)
+			(unlocked yes)
+			(layer "F.Fab")
+			(hide yes)
+			(effects
+				(font
+					(size 1 1)
+					(thickness 0.15)
+				)
+			)
+		)
 		(property ki_fp_filters "C_*")
 		(sheetname "/")
@@
 			)
 		)
+		(property "LCSC Part" "C19702"
+			(at 0 0 90)
+			(unlocked yes)
+			(layer "F.Fab")
+			(hide yes)
+			(effects
+				(font
+					(size 1 1)
+					(thickness 0.15)
+				)
+			)
+		)
 		(property ki_fp_filters "C_*")
 		(sheetname "/")
@@
 			)
 		)
+		(property "LCSC Part" "C19702"
+			(at 0 0 0)
+			(unlocked yes)
+			(layer "F.Fab")
+			(hide yes)
+			(effects
+				(font
+					(size 1 1)
+					(thickness 0.15)
+				)
+			)
+		)
 		(property ki_fp_filters "C_*")
 		(sheetname "/")
@@
 			(hide yes)
 			(effects
+				(font
+					(size 1 1)
+					(thickness 0.15)
+				)
+			)
+		)
+		(property "LCSC Part" "C19702"
+			(at 0 0 270)
+			(unlocked yes)
+			(layer "F.Fab")
+			(hide yes)
+			(effects
